File: Hardware/Eagle/2020-11-23 BOSS-RoboClaw-Interface.sch (EAGLE design)
At the start: 8 parts, among them IC1 ISO7221A, J2 PINHD-1X2-MOLEX-22112022, J3 Molex 22122034, X1 Amphenol L77SDAH15SOL2RM8C309

Commit message: Created schematic PDF and saved 2020-11-23 version
Parts:
- removed J4: (no value), AUmlib:FE10-2SAMTEC-ESW-110-44-S-D
- added J5: SAMTEC ESQ-110-33-T-D, AUmlib:PINHD-2X10-ESQ-110-33-T-DSAMTEC
- added J6: SAMTEC-ESQ-105-33-T-S, AUmlib:PINHD-1X5-ESQ-105-33-T-S
- IC1: value ISO7221A -> TI ISO7221ADR; device AUmlib:ISO7221A -> AUmlib:ISO7221ISO7221
- J1: value (none) -> MOLEX 22112022; device AUmlib:PINHD-2X2AMP-75869-130LF -> AUmlib:PINHD-1X2-MOLEX-22112022
- J2: value PINHD-1X2-MOLEX-22112022 -> MOLEX 22122034; device AUmlib:PINHD-1X2-MOLEX-22112022 -> AUmlib:PINHD-1X3RA-MOLEX-22122034
- J3: value Molex 22122034 -> Amphenol 75869-130LF; device AUmlib:PINHD-1X3RA-MOLEX-22122034 -> AUmlib:PINHD-2X2AMP-75869-130LF
Connections:
- removed net LIMIT/HOME: J3.1, J3.2
- removed net N$1: IC1.INA, J1.1
- removed net N$2: IC1.OUTB, J1.3
- new net LIMIT: J2.1, J2.2, J6.4
- new net RXMCU: IC1.OUTB, J3.3
- new net TXMCU: IC1.INA, J3.1
- net ENC1A: now also J5.8; no longer J4.7
- net ENC1B: now also J5.7; no longer J4.8
- net GND: now also J2.3, J5.15; no longer J3.3, J4.16
- net GND-ISO: now also J3.4; no longer J1.4
- net M1A: now also J1.1, X1-2.F; no longer J2.2, X1-9.F
- net M1B: now also J1.2, X1-9.F; no longer J2.1, X1-2.F
- net RX: now also J6.1
- net TX: now also J6.2
- net VCC1: now also J5.16; no longer J4.15
- net VCC2: now also J3.2; no longer J1.2
Other:
- note added: "Serial Isolator OUTA: RX RoboClaw INB: TX RoboClaw INA: Serial TX on MCU OUTB: Serial RX on MCU"
- note removed: "Next rev: Make bigger holes for the elevated sockets, check to see if pins 12 & 14 are grounds and if so, ground them and remove the vias"
- note removed: "Parts List One each except we need two 0.1uF bypass caps and four each nylon standoffs and nuts. D-SUB 15 Female, connects to PI M-227.10 motor, Amphenol L77SDAH15SOL2RM8C309, Digikey L77SDAH15SOL2RM8C309-ND 6-position clamp terminal (not shown, replace RoboClaw's screw terminal), Phoenix Contact 1823670, Digikey 277-11662-1-ND 3x10 socket (connects to RoboClaw pin headers, shown as SV1 and SV2),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"
- note removed: "Serial Isolator OUTA: RX RoboClaw INB: TX RoboClaw INA: Serial from MCU OUTB: Serial to MCU"
