File: Hardware/Eagle/2021-02-15 BOSS-RoboClaw-Interface.sch (EAGLE design)
At the start: 10 parts, among them IC1 ISO7221AQDRQ1, J1 MOLEX 22112024, J2 MOLEX 22122034, J3 Amphenol 75869-130LF, J5 SAMTEC ESQ-110-33-T-D, J6 SAMTEC-ESQ-105-33-T-S, X1 Amphenol L77SDAH15SOL2RM8C309

Commit message: Added pullup to limit switch line
Parts:
- removed R1: 10K, AUmlib:R-US_R0805
Connections:
- removed net ROBO-RX: IC1.OUTA, J6.1
- removed net ROBO0TX: IC1.INB, J6.2
- new net RXMCU: IC1.OUTB, J3.3
- new net TXMCU: IC1.INA, J3.1
- net LIMIT: no longer R1.1
- net RX: now also IC1.OUTA, J6.1; no longer IC1.INA, J3.1
- net TX: now also IC1.INB, J6.2; no longer IC1.OUTB, J3.3
- net VCC1: no longer R1.2
Other:
- moved on the sheet: J2, J6
